File: kicad/cp2102.sch (KiCad schematic (older format))
At the start: 10 parts, among them P1 CONN_01X05, P2 MICRO-USB-B, U1 CP2102

Commit message: ver2.0
Parts:
- added P3: CONN_01X05, BASIC:PIN_SOCKET_5, symbol CONN_01X05
- C1, C2, C3: footprint (none) -> BASIC:CAP_0603
- D1: footprint (none) -> BASIC:LED-0603; symbol LED -> LED-RESCUE-cp2102
- LOGO1: footprint (none) -> BASIC:LOGO_LEMBED
- LOGO2: footprint (none) -> BASIC:LOGO_SILK_OSHW_6x6mm
- P1: footprint (none) -> BASIC:PIN_SOCKET_5
- P2: footprint (none) -> BASIC:USB_B_MINI_SMD
- R1: footprint (none) -> BASIC:R_0603; symbol R -> R-RESCUE-cp2102
- U1: footprint (none) -> BASIC:QFN-28-1EP_5x5mm_Pitch0.5mm
Connections:
- net labels added: CTS, DSR, DTR, RTS
- wire segments 35 -> 45
- no-connect marks 9 -> 5
Other:
- moved on the sheet: C1, C2, C3, D1, LOGO1, LOGO2, P1, P2, R1, U1
